File: routageBE.sch (KiCad schematic (older format))
At the start: 50 parts, among them J1 Conn_01x03, J2 Conn_01x02, Q1 2N2907, Q10 BD138, Q11 TIP31, Q12 TIP32, Q13 2N2222, Q2 2N2907, Q3 2N2907, Q4 2N2907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

Commit message: schema sauf relay
Parts:
- removed U?: Jack_Mono, symbol BE-lib:Jack_Mono
- added U?: Jack_Mono, symbol BE-lib:Jack_Mono
Connections:
- net GND: now also U?.G
- net at C3.2: now also U?.T
Changed lines of the file:
@@
 $Comp
 L BE-lib:Jack_Mono U?
-U 1 1 5E7A268F
+U 1 1 5E79B849
 P 1800 3900
 F 0 "U?" H 1828 4167 50  0000 C CNN
